File: BADGE_LED_MATRIX_STM_MicroUSBALT/BadgeLedMatrix.brd (EAGLE design)
At the start: 100 x 50 mm, 110 parts, among them CN1 microUSB, IC1 STM32F0P, IC2 REG1117, Q1 12MHz, Q2 8MHz, U1 USBLC6SOT-23

Commit message: Speaker badge
Parts:
- removed JP1: USB-A-H, SparkFun-Connectors:USB-A-H
- added BATTERY: (no value), pinhead:1X02
Connections:
- new net N$5: BATTERY.1, S1.2
- net DMIN: no longer JP1.D-
- net DPLUS: no longer JP1.D+
- net GND: now also BATTERY.2; no longer JP1.GND
- net N$4: no longer S1.2
- net VIN: no longer JP1.VBUS
Routing:
- net N$5: track 0.00 -> 18.9 mm
- net VIN: track 39.7 -> 24.6 mm
- net DMIN: track 44.3 -> 39.8 mm, vias 3 -> 2
- net DPLUS: track 46.1 -> 42.1 mm
- net N$4: track 19.5 -> 15.9 mm
Other:
- board text added: "B+"
- board text added: "B-"
- board text added: "BATTERY"
- board text added: "HACKME"
- board text added: "OFF"
- board text added: "S P E A K E R"
- board text added: "To Program: 1. Connect to PC 2. Press & Hold Prog 3. Press & Release Reset 4. Release Reset"
- board text added: "WARNING: Do not exceed 5VDC battery Battery OFF before connect PC"
- board text removed: "P R O T O V 3"
- board text removed: "PROG"
- board text removed: "RUN"
- board text removed: "STM32F0"
- board text removed: "To Program: 1. Connect to PC 2. Slide to PROG 3. Press Reset"
