File: BADGE_LED_MATRIX_STM_MicroUSBALT/BadgeLedMatrix.brd (EAGLE design)
At the start: 100 x 50 mm, 110 parts, among them CN1 microUSB, IC1 STM32F0P, IC2 REG1117, Q1 12MHz, Q2 8MHz, U1 USBLC6SOT-23

Commit message: Updating for participant
Parts:
- C4, C6: device SparkFun-Capacitors:0805 -> SparkFun-Passives:0603-CAP
- moved C4 0.08 mm to (8.18, 47.0)
Other:
- board text added: "P A R T I C I P A N T"
- board text added: "To Program: 1. Connect to PC 2. Press & Hold Prog 3. Press & Release Reset"
- board text removed: "S P E A K E R"
- board text removed: "To Program: 1. Connect to PC 2. Press & Hold Prog 3. Press & Release Reset 4. Release Reset"
Changed lines of the file:
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@@
 <?xml version="1.0" encoding="utf-8"?>
 <!DOCTYPE eagle SYSTEM "eagle.dtd">
-<eagle version="7.5.0">
+<eagle version="7.6.0">
 <drawing>
 <settings>
@@
 <layers>
 <layer number="1" name="Top" color="4" fill="1" visible="yes" active="yes"/>
-<layer number="16" name="Bottom" color="1" fill="1" visible="yes" active="yes"/>
+<layer number="16" name="Bottom" color="1" fill="1" visible="no" active="yes"/>
 <layer number="17" name="Pads" color="2" fill="1" visible="yes" active="yes"/>
 <layer number="18" name="Vias" color="2" fill="1" visible="yes" active="yes"/>
@@
 <layer number="22" name="bPlace" color="7" fill="1" visible="yes" active="yes"/>
 <layer number="23" name="tOrigins" color="15" fill="1" visible="yes" active="yes"/>
-<layer number="24" name="bOrigins" color="15" fill="1" visible="yes" active="yes"/>
+<layer number="24" name="bOrigins" color="15" fill="1" visible="no" active="yes"/>
 <layer number="25" name="tNames" color="7" fill="1" visible="yes" active="yes"/>
-<layer number="26" name="bNames" color="7" fill="1" visible="yes" active="yes"/>
+<layer number="26" name="bNames" color="7" fill="1" visible="no" active="yes"/>
 <layer number="27" name="tValues" color="7" fill="1" visible="yes" active="yes"/>
-<layer number="28" name="bValues" color="7" fill="1" visible="yes" active="yes"/>
+<layer number="28" name="bValues" color="7" fill="1" visible="no" active="yes"/>
 <layer number="29" name="tStop" color="7" fill="3" visible="no" active="yes"/>
 <layer number="30" name="bStop" color="7" fill="6" visible="no" active="yes"/>
@@
 <circle x="41.91" y="26.67" radius="3.175" width="0.8128" layer="21"/>
 <circle x="34.29" y="17.145" radius="3.175" width="0.8128" layer="21"/>
-<text x="90.76205625" y="2.09595" size="4" layer="21" rot="SR270" align="top-right">S
+<text x="91.249109375" y="2.09595" size="3" layer="21" rot="SR270" align="top-right">P
+A
+R
+T
+I
+C
+I
 P
-E
 A
-K
-E
-R</text>
-<wire x1="44" y1="6.985" x2="89.992928125" y2="6.985" width="0.3048" layer="21"/>
+N
+T</text>
+<wire x1="40.843625" y1="6.985" x2="89.992928125" y2="6.985" width="0.3048" layer="21"/>
 <wire x1="89.992928125" y1="6.985" x2="92.71" y2="5.002125" width="0.3048" layer="21" curve="-72.242726"/>
 <wire x1="92.71" y1="5.002125" x2="92.70945" y2="0.638475" width="0.3048" layer="21"/>
@@
 <text x="34.5" y="33.5" size="1.778" layer="22" rot="MR180">OFF</text>
 <text x="10.5" y="13" size="1.778" layer="21">CH340G</text>
-<text x="2.5" y="32" size="2.1844" layer="21" rot="SR270">HACKME</text>
-<text x="58.5" y="4" size="2.1844" layer="22" rot="SMR0">To Program:
+<text x="1.404275" y="34.07146875" size="3" layer="21" rot="SR270">HACKME</text>
+<text x="58.616928125" y="6.16516875" size="2.1844" layer="22" rot="SMR0">To Program:
 1. Connect to PC
 2. Press &amp; Hold Prog
-3. Press &amp; Release Reset
-4. Release Reset</text>
+3. Press &amp; Release Reset</text>
 <wire x1="44.094878125" y1="31" x2="32.60555" y2="31" width="0.4064" layer="22"/>
 <wire x1="32.60555" y1="31" x2="29" y2="34.60555" width="0.4064" layer="22" curve="-90"/>
@@
 - Battery OFF before
   connect PC</text>
-<wire x1="49" y1="6.9" x2="49" y2="5" width="0.3048" layer="21"/>
-<wire x1="49" y1="5" x2="44.5" y2="0.5" width="0.3048" layer="21"/>
-<wire x1="48" y1="6.9" x2="48" y2="5" width="0.3048" layer="21"/>
-<wire x1="48" y1="5" x2="43.5" y2="0.5" width="0.3048" layer="21"/>
-<wire x1="47" y1="6.9" x2="47" y2="5" width="0.3048" layer="21"/>
-<wire x1="47" y1="5" x2="42.5" y2="0.5" width="0.3048" layer="21"/>
-<wire x1="46" y1="6.9" x2="46" y2="5" width="0.3048" layer="21"/>
-<wire x1="46" y1="5" x2="41.5" y2="0.5" width="0.3048" layer="21"/>
-<wire x1="45" y1="6.9" x2="45" y2="5" width="0.3048" layer="21"/>
-<wire x1="45" y1="5" x2="40.5" y2="0.5" width="0.3048" layer="21"/>
 <wire x1="44" y1="6.938578125" x2="44" y2="5" width="0.3048" layer="21"/>
 <wire x1="44" y1="5" x2="39.5" y2="0.5" width="0.3048" layer="21"/>
+<text x="27.337096875" y="23.17790625" size="1.778" layer="21" rot="MR180">B+</text>
+<text x="27.147259375" y="15.539671875" size="1.778" layer="21" rot="MR180">B-</text>
+<wire x1="42.985675" y1="6.938578125" x2="42.985675" y2="5" width="0.3048" layer="21"/>
+<wire x1="42.985675" y1="5" x2="38.485675" y2="0.612790625" width="0.3048" layer="21"/>
+<wire x1="41.858646875" y1="6.938578125" x2="41.858646875" y2="5" width="0.3048" layer="21"/>
+<wire x1="41.858646875" y1="5" x2="37.358646875" y2="0.584590625" width="0.3048" layer="21"/>
+<wire x1="40.844321875" y1="6.938578125" x2="40.844321875" y2="5" width="0.3048" layer="21"/>
+<wire x1="40.844321875" y1="5" x2="36.344321875" y2="0.69738125" width="0.3048" layer="21"/>
 </plain>
 <attributes>
@@
 <attribute name="VALUE" x="16.779" y="39.497" size="1.27" layer="27" ratio="10" rot="R180"/>
 </element>
-<element name="C4" library="SparkFun-Capacitors" package="0805" value="10uf" x="8.255" y="46.99" rot="R90">
-<attribute name="PROD_ID" value="CAP-08402" x="4.445" y="25.4" size="1.778" layer="27" rot="R90" display="off"/>
-</element>
 <element name="C5" library="SparkFun-Passives" package="0603-CAP" value=".1uf" x="5.715" y="46.99" rot="R90"/>
-<element name="C6" library="SparkFun-Capacitors" package="0805" value="10uf" x="13.97" y="46.99" rot="R90">
-<attribute name="PROD_ID" value="CAP-08402" x="0" y="31.75" size="1.778" layer="27" rot="R90" display="off"/>
-</element>
 <element name="C7" library="SparkFun-Passives" package="0603-CAP" value=".1uf" x="11.43" y="46.99" rot="R90"/>
 <element name="IC1" library="digital-ic" package="TSSOP20" value="STM32F0P" x="22.86" y="27.94" smashed="yes" rot="R180">
@@
 <element name="CN1" library="microbuilder" package="4UCONN_20329" value="microUSB" x="4.3" y="39.5" smashed="yes" rot="MR90"/>
 <element name="BATTERY" library="pinhead" package="1X02" value="" x="28.5" y="18.5" rot="MR270"/>
+<element name="C6" library="SparkFun-Passives" package="0603-CAP" value="10uf" x="13.985775" y="47.0119625" rot="R90"/>
+<element name="C4" library="SparkFun-Passives" package="0603-CAP" value="10uf" x="8.17815625" y="46.962475" rot="R90"/>
 </elements>
 <signals>
@@
 <contactref element="C1" pad="2"/>
 <contactref element="CH340G" pad="1"/>
-<contactref element="IC2" pad="1"/>
-<contactref element="IC2" pad="1"/>
-<contactref element="C4" pad="2"/>
 <contactref element="C5" pad="2"/>
-<contactref element="C6" pad="2"/>
 <contactref element="C7" pad="2"/>
 <contactref element="C9" pad="2"/>
@@
 <contactref element="ROWS" pad="13"/>
 <contactref element="ROWS" pad="8"/>
-<contactref element="COLUMNS" pad="8"/>
-<contactref element="COLUMNS" pad="8"/>
 <polygon width="0.6096" layer="1">
 <vertex x="0" y="0"/>
@@
 <contactref element="RESET" pad="2"/>
 <contactref element="ST-LINK" pad="3"/>
-<contactref element="COLUMNS" pad="13"/>
 <contactref element="U1" pad="2"/>
 <contactref element="IC1" pad="15"/>
@@
 <wire x1="5.2" y1="40.925" x2="5.075" y2="40.8" width="0.4064" layer="16"/>
 <contactref element="BATTERY" pad="2"/>
+<contactref element="IC2" pad="1"/>
+<contactref element="COLUMNS" pad="8"/>
+<contactref element="COLUMNS" pad="13"/>
+<contactref element="C6" pad="2"/>
+<contactref element="C4" pad="2"/>
 </signal>
 <signal name="VCC">
 <contactref element="IC2" pad="2"/>
 <contactref element="C7" pad="1"/>
-<contactref element="C6" pad="1"/>
 <contactref element="CH340G" pad="16"/>
 <via x="40.005" y="19.05" extent="1-16" drill="0.8" diameter="0.6096"/>
@@
 <via x="17.145" y="19.05" extent="1-16" drill="0.8"/>
 <contactref element="CH340G" pad="4"/>
-<wire x1="11.43" y1="46.14" x2="13.92" y2="46.14" width="0.8128" layer="1"/>
-<wire x1="13.92" y1="46.14" x2="13.97" y2="46.09" width="0.8128" layer="1"/>
 <wire x1="17.145" y1="44.45" x2="15.875" y2="46.09" width="0.8128" layer="1"/>
-<wire x1="15.875" y1="46.09" x2="13.97" y2="46.09" width="0.8128" layer="1"/>
 <wire x1="15.875" y1="10.922" x2="15.875" y2="17.145" width="0.8128" layer="1"/>
 <wire x1="15.875" y1="17.145" x2="16.185" y2="17.61" width="0.8128" layer="1"/>
@@
 <wire x1="13.3246" y1="41.8846" x2="13.3246" y2="44.2454" width="0.8128" layer="1"/>
 <wire x1="13.3246" y1="44.2454" x2="11.43" y2="46.14" width="0.8128" layer="1"/>
+<contactref element="C6" pad="1"/>
+<wire x1="13.985775" y1="46.1619625" x2="15.8030375" y2="46.1619625" width="0.8128" layer="1"/>
+<wire x1="15.8030375" y1="46.1619625" x2="15.875" y2="46.09" width="0.8128" layer="1"/>
+<wire x1="13.9638125" y1="46.14" x2="13.985775" y2="46.1619625" width="0.8128" layer="1"/>
+<wire x1="13.9638125" y1="46.14" x2="13.9638125" y2="44.8846125" width="0.8128" layer="1"/>
+<wire x1="13.9638125" y1="44.8846125" x2="13.3246" y2="44.2454" width="0.8128" layer="1"/>
 </signal>
 <signal name="C0">
@@
 <signal name="VIN">
 <contactref element="IC2" pad="3"/>
-<contactref element="C4" pad="1"/>
 <contactref element="C5" pad="1"/>
 <wire x1="9.525" y1="40.371" x2="9.525" y2="36.52" width="0.8128" layer="1"/>
 <wire x1="5.715" y1="46.14" x2="8.205" y2="46.14" width="0.8128" layer="1"/>
-<wire x1="8.205" y1="46.14" x2="8.255" y2="46.09" width="0.8128" layer="1"/>
 <via x="6.35" y="33.02" extent="1-16" drill="0.6"/>
 <wire x1="6.35" y1="33.02" x2="9.525" y2="36.52" width="0.8128" layer="1"/>
 <contactref element="CN1" pad="VBUS"/>
 <wire x1="11.0386" y1="41.8846" x2="11.0386" y2="43.3064" width="0.8128" layer="1"/>
-<wire x1="11.0386" y1="43.3064" x2="8.255" y2="46.09" width="0.8128" layer="1"/>
 <wire x1="9.525" y1="40.371" x2="11.0386" y2="41.8846" width="0.8128" layer="1"/>
 <wire x1="5.075" y1="38.2" x2="5.3" y2="38.2" width="0.4064" layer="16"/>
@@
 <wire x1="6.5" y1="33.17" x2="6.35" y2="33.02" width="0.4064" layer="16"/>
 <wire x1="5.3" y1="38.2" x2="6.5" y2="37" width="0.4064" layer="16"/>
+<contactref element="C4" pad="1"/>
+<wire x1="8.205" y1="46.14" x2="11.0386" y2="43.3064" width="0.8128" layer="1"/>
+<wire x1="8.205" y1="46.14" x2="8.17815625" y2="46.112475" width="0" layer="19" extent="1-1"/>
 </signal>
 <signal name="OVERFLOW">
