File: BADGE_LED_MATRIX_STM_MicroUSBALT/BadgeLedMatrix.sch (EAGLE design)
At the start: 106 parts, among them CN1 microUSB, IC1 STM32F0P, IC2 REG1117, Q1 12MHz, Q2 8MHz, U1 USBLC6SOT-23

Commit message: Speaker badge
Parts:
- removed JP1: USB-A-H, SparkFun-Connectors:USB-A-H
- added BATTERY: (no value), pinhead:PINHD-1X2
Connections:
- new net N$5: BATTERY.1, S1.P
- net DMIN: no longer JP1.D-
- net DPLUS: no longer JP1.D+
- net GND: now also BATTERY.2; no longer JP1.GND
- net N$4: no longer S1.P
- net VIN: no longer JP1.VBUS
Changed lines of the file:
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@@
 <part name="CH340G" library="digital-ic" deviceset="CH340G" device="CH340G"/>
 <part name="SUPPLY2" library="supply2" deviceset="GND" device=""/>
-<part name="JP1" library="SparkFun-Connectors" deviceset="USB" device="-A-H"/>
 <part name="SUPPLY3" library="supply2" deviceset="GND" device=""/>
 <part name="GND14" library="supply1" deviceset="GND" device=""/>
@@
 <part name="CN1" library="microbuilder" deviceset="USB" device="MICRO_20329" value="microUSB"/>
 <part name="SUPPLY10" library="supply2" deviceset="GND" device=""/>
+<part name="BATTERY" library="pinhead" deviceset="PINHD-1X2" device=""/>
+<part name="SUPPLY11" library="supply2" deviceset="GND" device=""/>
 </parts>
 <sheets>
@@
 <instance part="CH340G" gate="G$1" x="464.82" y="185.42"/>
 <instance part="SUPPLY2" gate="GND" x="454.66" y="195.58" rot="R180"/>
-<instance part="JP1" gate="G$1" x="414.02" y="193.04"/>
 <instance part="SUPPLY3" gate="GND" x="406.4" y="193.04" rot="R270"/>
 <instance part="GND14" gate="1" x="259.08" y="215.9"/>
@@
 <instance part="CN1" gate="G$1" x="401.32" y="170.18"/>
 <instance part="SUPPLY10" gate="GND" x="416.56" y="165.1" rot="R90"/>
+<instance part="BATTERY" gate="G$1" x="381" y="325.12"/>
+<instance part="SUPPLY11" gate="GND" x="368.3" y="320.04"/>
 </instances>
 <busses>
@@
 </segment>
 <segment>
-<pinref part="JP1" gate="G$1" pin="GND"/>
 <wire x1="411.48" y1="193.04" x2="408.94" y2="193.04" width="0.1524" layer="91"/>
 <pinref part="SUPPLY3" gate="GND" pin="GND"/>
@@
 <wire x1="414.02" y1="165.1" x2="411.48" y2="165.1" width="0.1524" layer="91"/>
 </segment>
+<segment>
+<pinref part="BATTERY" gate="G$1" pin="2"/>
+<pinref part="SUPPLY11" gate="GND" pin="GND"/>
+<wire x1="378.46" y1="325.12" x2="368.3" y2="325.12" width="0.1524" layer="91"/>
+<wire x1="368.3" y1="325.12" x2="368.3" y2="322.58" width="0.1524" layer="91"/>
+<junction x="368.3" y="322.58"/>
+<junction x="378.46" y="325.12"/>
+</segment>
 </net>
 <net name="DPLUS" class="0">
 <segment>
-<pinref part="JP1" gate="G$1" pin="D+"/>
 <wire x1="411.48" y1="200.66" x2="403.86" y2="200.66" width="0.1524" layer="91"/>
 <label x="401.32" y="200.66" size="1.778" layer="95"/>
@@
 <net name="DMIN" class="0">
 <segment>
-<pinref part="JP1" gate="G$1" pin="D-"/>
 <wire x1="411.48" y1="198.12" x2="403.86" y2="198.12" width="0.1524" layer="91"/>
 <label x="401.32" y="198.12" size="1.778" layer="95"/>
@@
 </segment>
 <segment>
-<pinref part="JP1" gate="G$1" pin="VBUS"/>
 <wire x1="411.48" y1="195.58" x2="403.86" y2="195.58" width="0.1524" layer="91"/>
 <label x="401.32" y="195.58" size="1.778" layer="95"/>
@@
 <junction x="353.06" y="314.96"/>
 <pinref part="PRG" gate="G$1" pin="2"/>
-<wire x1="353.06" y1="325.12" x2="353.06" y2="314.96" width="0.1524" layer="91"/>
-<pinref part="S1" gate="1" pin="P"/>
-<wire x1="347.98" y1="325.12" x2="353.06" y2="325.12" width="0.1524" layer="91"/>
 </segment>
 </net>
@@
 </segment>
 </net>
+<net name="N$5" class="0">
+<segment>
+<pinref part="BATTERY" gate="G$1" pin="1"/>
+<wire x1="378.46" y1="327.66" x2="358.14" y2="327.66" width="0.1524" layer="91"/>
+<wire x1="358.14" y1="327.66" x2="358.14" y2="325.12" width="0.1524" layer="91"/>
+<pinref part="S1" gate="1" pin="P"/>
+<wire x1="358.14" y1="325.12" x2="347.98" y2="325.12" width="0.1524" layer="91"/>
+<junction x="347.98" y="325.12"/>
+<junction x="378.46" y="327.66"/>
+</segment>
+</net>

Commit message: Updating for participant
Parts:
- C4, C6: device SparkFun-Capacitors:22UF-6.3V-20%(0805) -> SparkFun-Passives:CAP0603-CAP
Changed lines of the file:
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@@
 <?xml version="1.0" encoding="utf-8"?>
 <!DOCTYPE eagle SYSTEM "eagle.dtd">
-<eagle version="7.5.0">
+<eagle version="7.6.0">
 <drawing>
 <settings>
@@
 <part name="GND5" library="supply1" deviceset="GND" device=""/>
 <part name="GND20" library="supply1" deviceset="GND" device=""/>
-<part name="C4" library="SparkFun-Capacitors" deviceset="22UF-6.3V-20%(0805)" device="" value="10uf"/>
 <part name="C5" library="SparkFun-Passives" deviceset="CAP" device="0603-CAP" value=".1uf"/>
-<part name="C6" library="SparkFun-Capacitors" deviceset="22UF-6.3V-20%(0805)" device="" value="10uf"/>
 <part name="C7" library="SparkFun-Passives" deviceset="CAP" device="0603-CAP" value=".1uf"/>
 <part name="GND3" library="supply1" deviceset="GND" device=""/>
@@
 <part name="IC1" library="digital-ic" deviceset="STM32F0*" device="P"/>
 <part name="SUPPLY5" library="supply2" deviceset="GND" device=""/>
-<part name="SUPPLY6" library="supply2" deviceset="GND" device=""/>
 <part name="Q2" library="crystal" deviceset="CRYSTAL" device="HC49U70" value="8MHz"/>
 <part name="C8" library="SparkFun-Capacitors" deviceset="CAP" device="0603-CAP" value="22pF"/>
@@
 <part name="BATTERY" library="pinhead" deviceset="PINHD-1X2" device=""/>
 <part name="SUPPLY11" library="supply2" deviceset="GND" device=""/>
+<part name="GND2" library="supply1" deviceset="GND" device=""/>
+<part name="C6" library="SparkFun-Passives" deviceset="CAP" device="0603-CAP" value="10uf"/>
+<part name="C4" library="SparkFun-Passives" deviceset="CAP" device="0603-CAP" value="10uf"/>
 </parts>
 <sheets>
@@
 <instance part="GND5" gate="1" x="233.68" y="218.44"/>
 <instance part="GND20" gate="1" x="274.32" y="218.44"/>
-<instance part="C4" gate="G$1" x="233.68" y="226.06"/>
 <instance part="C5" gate="G$1" x="243.84" y="226.06"/>
-<instance part="C6" gate="G$1" x="274.32" y="226.06"/>
 <instance part="C7" gate="G$1" x="284.48" y="226.06"/>
 <instance part="GND3" gate="1" x="243.84" y="218.44"/>
@@
 <instance part="IC1" gate="G$1" x="381" y="279.4"/>
 <instance part="SUPPLY5" gate="GND" x="436.88" y="226.06"/>
-<instance part="SUPPLY6" gate="GND" x="439.42" y="264.16"/>
 <instance part="Q2" gate="G$1" x="342.9" y="294.64"/>
 <instance part="C8" gate="G$1" x="337.82" y="287.02"/>
@@
 <instance part="BATTERY" gate="G$1" x="381" y="325.12"/>
 <instance part="SUPPLY11" gate="GND" x="368.3" y="320.04"/>
+<instance part="GND2" gate="1" x="441.96" y="264.16"/>
+<instance part="C6" gate="G$1" x="274.32" y="226.06"/>
+<instance part="C4" gate="G$1" x="233.68" y="226.06"/>
 </instances>
 <busses>
@@
 </segment>
 <segment>
-<pinref part="IC2" gate="G$1" pin="GND"/>
-<pinref part="GND14" gate="1" pin="GND"/>
-<wire x1="259.08" y1="220.98" x2="259.08" y2="218.44" width="0.1524" layer="91"/>
-</segment>
-<segment>
-<pinref part="C4" gate="G$1" pin="2"/>
 <pinref part="GND5" gate="1" pin="GND"/>
 <wire x1="233.68" y1="223.52" x2="233.68" y2="220.98" width="0.1524" layer="91"/>
+<pinref part="C4" gate="G$1" pin="2"/>
 </segment>
 <segment>
@@
 </segment>
 <segment>
-<pinref part="C6" gate="G$1" pin="2"/>
 <pinref part="GND20" gate="1" pin="GND"/>
 <wire x1="274.32" y1="223.52" x2="274.32" y2="220.98" width="0.1524" layer="91"/>
+<pinref part="C6" gate="G$1" pin="2"/>
 </segment>
 <segment>
@@
 <pinref part="SUPPLY5" gate="GND" pin="GND"/>
 <wire x1="444.5" y1="228.6" x2="436.88" y2="228.6" width="0.1524" layer="91"/>
-</segment>
-<segment>
-<pinref part="SUPPLY6" gate="GND" pin="GND"/>
-<pinref part="COLUMNS" gate="A" pin="GND"/>
-<pinref part="COLUMNS" gate="A" pin="G"/>
-<wire x1="441.96" y1="271.78" x2="439.42" y2="269.24" width="0.1524" layer="91"/>
-<wire x1="439.42" y1="269.24" x2="439.42" y2="266.7" width="0.1524" layer="91"/>
-<wire x1="439.42" y1="266.7" x2="441.96" y2="266.7" width="0.1524" layer="91"/>
-<junction x="439.42" y="266.7"/>
 </segment>
 <segment>
@@
 <junction x="378.46" y="325.12"/>
 </segment>
+<segment>
+<pinref part="IC2" gate="G$1" pin="GND"/>
+<pinref part="GND14" gate="1" pin="GND"/>
+<wire x1="259.08" y1="218.44" x2="259.08" y2="220.98" width="0.1524" layer="91"/>
+</segment>
+<segment>
+<pinref part="COLUMNS" gate="A" pin="GND"/>
+<pinref part="GND2" gate="1" pin="GND"/>
+<pinref part="COLUMNS" gate="A" pin="G"/>
+<wire x1="441.96" y1="271.78" x2="441.96" y2="266.7" width="0.1524" layer="91"/>
+<junction x="441.96" y="271.78"/>
+<junction x="441.96" y="266.7"/>
+</segment>
 </net>
 <net name="DPLUS" class="0">
@@
 <label x="228.6" y="236.22" size="1.778" layer="95"/>
 <wire x1="228.6" y1="233.68" x2="233.68" y2="233.68" width="0.1524" layer="91"/>
-<pinref part="C4" gate="G$1" pin="1"/>
 <wire x1="233.68" y1="233.68" x2="243.84" y2="233.68" width="0.1524" layer="91"/>
 <wire x1="243.84" y1="233.68" x2="246.38" y2="233.68" width="0.1524" layer="91"/>
@@
 <wire x1="243.84" y1="231.14" x2="243.84" y2="233.68" width="0.1524" layer="91"/>
 <junction x="243.84" y="233.68"/>
+<pinref part="C4" gate="G$1" pin="1"/>
 </segment>
 <segment>
@@
 <wire x1="284.48" y1="231.14" x2="284.48" y2="233.68" width="0.1524" layer="91"/>
 <junction x="284.48" y="233.68"/>
-<pinref part="C6" gate="G$1" pin="1"/>
 <wire x1="274.32" y1="231.14" x2="274.32" y2="233.68" width="0.1524" layer="91"/>
 <junction x="274.32" y="233.68"/>
 <label x="289.56" y="236.22" size="1.778" layer="95"/>
-</segment>
-<segment>
+<pinref part="C6" gate="G$1" pin="1"/>
+</segment>
+<segment>
